File: adf5355/adf5355.sch (KiCad schematic (older format))
At the start: 86 parts, among them J1 REF_IN_A, J2 RF_B, J3 RF_A_P, J4 REF_IN_B, J5 RF_A_N, J6 Conn_01x02_Male, J7 Conn_01x10_Male, U1 L7806, U2 ADM7150, U3 ADM7150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

Commit message: Placing more components
Parts:
- added C5, C58: 1u, Capacitors_SMD:C_0603, symbol Device:C
- added C56, C60: 100p, Capacitors_SMD:C_0603, symbol Device:C
- added C57, C61: 10p, Capacitors_SMD:C_0603, symbol Device:C
- added C59, C7: 10n, Capacitors_SMD:C_0603, symbol Device:C
- added L4, L5: L, Capacitors_SMD:C_0805_HandSoldering, symbol Device:L
- C14, C15, C20, C26, C29, C31, C32, C38, C48, C51, C54, C9: footprint Capacitors_SMD:C_0805 -> Capacitors_SMD:C_0603
- C30, C55: footprint Capacitors_SMD:C_1206 -> Capacitors_SMD:C_0603
- C47, C52: footprint Capacitors_SMD:C_1812 -> Capacitors_SMD:C_0603
Connections:
- wire segments 241 -> 269
Other:
- moved on the sheet: C6
