File: adf5355/_saved_adf5355.sch (KiCad schematic (older format))
At the start: 96 parts, among them J1 REF_IN_A, J2 RF_B, J3 RF_A_P, J4 REF_IN_B, J5 RF_A_N, J6 Conn_01x02_Male, J7 Conn_01x10_Male, U1 L7806, U2 ADM7150, U3 ADM7150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

Commit message: More placing
Parts:
- R13: footprint Resistors_SMD:R_0805 -> Resistors_SMD:R_0603
Changed lines of the file:
@@
 F 0 "R13" H 7430 4804 50  0000 R CNN
 F 1 "220" H 7430 4895 50  0000 R CNN
-F 2 "Resistors_SMD:R_0805" V 7430 4850 50  0001 C CNN
+F 2 "Resistors_SMD:R_0603" V 7430 4850 50  0001 C CNN
 F 3 "~" H 7500 4850 50  0001 C CNN
 	1    7500 4850
