File: adf_arduino_adapter/adf_arduino_adapter/adf_arduino_adapter.kicad_pcb (KiCad board)
At the start: 2 copper layers, 14 parts, among them J1 Conn_01x10_Female

Commit message: more frac n
Parts:
- moved R12 42.5 mm to (153.7, 69.7), turned to 270 degrees
- moved J1 41.2 mm to (144.4, 117.6), turned to 0 degrees
- moved R9 37.3 mm to (158.2, 69.7), turned to 270 degrees
- moved R1 31.6 mm to (144.9, 110.7), turned to 90 degrees
- moved R10 31.2 mm to (158.6, 92.5), turned to 270 degrees
- moved R11 31.1 mm to (161.2, 69.7), turned to 270 degrees
- moved R7 30.5 mm to (152.5, 73.7)
- moved R8 29.2 mm to (161.2, 92.5), turned to 270 degrees
- moved R2 26.3 mm to (151.5, 110.7), turned to 90 degrees
- moved R5 21.3 mm to (160.2, 76.2), turned to 0 degrees
- moved R4 19.9 mm to (160.1, 96.5), turned to 0 degrees
- moved R3 19.8 mm to (160.1, 99.1), turned to 0 degrees
- moved R6 19.0 mm to (160.0, 73.7), turned to 0 degrees
Routing:
- net Net-(A1-Pad16): track 53.2 -> 2.41 mm
- net GND: track 19.4 -> 69.8 mm
- net /CE: track 9.72 -> 59.7 mm
- net Net-(A1-Pad14): track 42.9 -> 2.16 mm
- net /DATA: track 10.2 -> 49.6 mm
- net /CLK: track 10.2 -> 46.9 mm
- net Net-(A1-Pad30): track 33.7 -> 6.60 mm
- net /LE: track 10.2 -> 26.7 mm
- net Net-(A1-Pad5): track 18.5 -> 2.23 mm
- net Net-(A1-Pad6): track 18.0 -> 2.29 mm
- net /MUX: track 10.2 -> 25.7 mm
- net Net-(A1-Pad15): track 15.1 -> 2.36 mm
Other:
- board outline added: 27.9 x 52.8 mm
